File: Raspberry-Pi-Hat/Raspberry-Pi-Hat.kicad_pcb (KiCad board)
At the start: 2 copper layers, 65 x 56 mm, 74 parts, among them J1 Screw_Terminal_01x04, J2 Screw_Terminal_01x02, J3 40HAT, J4 Screw_Terminal_01x02, J5 Screw_Terminal_01x04, J9 CONN_01X02, M1 Fan_Tacho_PWM, Q1 DMG2305UX, Q2 DMMT5401, U1 ADM3490ExR, U2 CAT24C32, U3 TCAN330, U4 LMZ13608, U5 AB0805, U6 MCP2515-xSO, U7 TXB0102DCU, Y1 32.768 kHz, Y2 8MHz

Commit message: Finalisation of the Project
Correcte last problems
Create gerber files
Parts:
- added G***: LOGO, project_footprints:Mimosa-Logo, B.Cu at (98.1, 102.2)
- added REF**: OSHW-Logo2_9.8x8mm_SilkScreen, Symbol:OSHW-Logo2_9.8x8mm_SilkScreen, B.Cu at (134.3, 104.5)
- C1: footprint Capacitor_SMD:C_1206_3216Metric_Pad1.42x1.75mm_HandSolder -> Capacitor_SMD:CP_Elec_10x12.5; moved to F.Cu
- C11, C12, C13, C5, C7, D1, R1, R12, R13, R15, R2, U3: moved to B.Cu
- moved C1 12.7 mm to (122.9, 94.7), turned to 270 degrees
- moved C11 12.7 mm to (109.8, 100.4), turned to 90 degrees
- moved R1 8.12 mm to (126.2, 94.0), turned to 90 degrees
- moved C13 8.00 mm to (116.3, 96.8)
- moved R12 7.49 mm to (112.5, 100.4), turned to 270 degrees
- moved C5 5.56 mm to (128.9, 94.0), turned to 270 degrees
- moved C7 3.19 mm to (128.8, 99.2), turned to 270 degrees
- moved R2 3.06 mm to (122.8, 95.0)
- moved R15 3.03 mm to (130.9, 88.9), turned to 0 degrees
- moved C12 2.99 mm to (117.8, 100.4), turned to 270 degrees
- moved D1 2.89 mm to (123.3, 108.2), turned to 270 degrees
- moved U3 2.72 mm to (123.2, 98.6)
- moved C8 2.60 mm to (97.1, 98.2)
- moved R13 2.29 mm to (115.2, 100.4), turned to 270 degrees
- moved U1 1.57 mm to (102.3, 97.8)
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Routing:
- net Net-(C11-Pad1): track 23.3 -> 32.9 mm
- net +12V: track 56.7 -> 65.0 mm
- net TX_CAN: track 19.6 -> 12.9 mm, vias 2 -> 1
- net GND: track 11.0 -> 14.9 mm, vias 0 -> 10
- net Net-(C12-Pad2): track 29.4 -> 25.5 mm
- net Net-(R2-Pad1): track 2.79 -> 6.28 mm
- net +3V3: track 156.4 -> 159.7 mm, vias 4 -> 5
- net /FAN-RPM-(GPIO24): track 59.5 -> 61.5 mm
- net Net-(J1-Pad2): track 18.9 -> 20.7 mm
- net +5V: track 141.9 -> 143.7 mm
- net TX_NMEA183: track 43.9 -> 42.2 mm
- net Net-(J1-Pad4): track 19.4 -> 21.0 mm
- net Net-(J1-Pad1): track 18.6 -> 20.2 mm
- net Net-(J1-Pad3): track 18.5 -> 20.0 mm
- net Net-(R14-Pad2): track 6.22 -> 7.66 mm, vias 0 -> 1
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Other:
- board text added: "Mimosa - Power Hat - V0 Designed by Jérôme Béguin 08.2020"
