File: Raspberry-Pi-Hat/Raspberry-Pi-Hat.sch (KiCad schematic (older format))
At the start: 74 parts, among them J1 Screw_Terminal_01x04, J2 Screw_Terminal_01x02, J3 40HAT, J4 Screw_Terminal_01x02, J5 Screw_Terminal_01x04, J9 CONN_01X02, M1 Fan_Tacho_PWM, Q1 DMG2305UX, Q2 DMMT5401, U1 ADM3490ExR, U2 CAT24C32, U3 TCAN330, U4 LMZ13608, U5 AB0805, U6 MCP2515-xSO, U7 TXB0102DCU, Y1 32.768 kHz, Y2 8MHz

Commit message: All 3d model included
Parts:
- J1, J5: footprint Connector_Phoenix_MSTB:PhoenixContact_MSTBVA_2,5_4-G-5,08_1x04_P5.08mm_Vertical -> TerminalBlock_Phoenix:TerminalBlock_Phoenix_MKDS-3-4-5.08_1x04_P5.08mm_Horizontal
- J2, J4: footprint Connector_Phoenix_MSTB:PhoenixContact_MSTBVA_2,5_2-G-5,08_1x02_P5.08mm_Vertical -> TerminalBlock_Phoenix:TerminalBlock_Phoenix_MKDS-3-2-5.08_1x02_P5.08mm_Horizontal
- U2: footprint Package_SOIC:SOIC-8_3.9x4.9mm_P1.27mm -> Package_SO:SOIC-8_3.9x4.9mm_P1.27mm
Changed lines of the file:
@@
 F 0 "U2" H 2450 6200 50  0000 C CNN
 F 1 "CAT24C32" H 1850 6200 50  0000 C CNN
-F 2 "Package_SOIC:SOIC-8_3.9x4.9mm_P1.27mm" H 2100 5850 50  0001 C CNN
+F 2 "Package_SO:SOIC-8_3.9x4.9mm_P1.27mm" H 2100 5850 50  0001 C CNN
 F 3 "" H 2100 5850 50  0000 C CNN
 	1    2100 5850
@@
 F 0 "J4" H 14680 842 50  0000 L CNN
 F 1 "Screw_Terminal_01x02" H 14680 751 50  0000 L CNN
-F 2 "Connector_Phoenix_MSTB:PhoenixContact_MSTBVA_2,5_2-G-5,08_1x02_P5.08mm_Vertical" H 14600 850 50  0001 C CNN
+F 2 "TerminalBlock_Phoenix:TerminalBlock_Phoenix_MKDS-3-2-5.08_1x02_P5.08mm_Horizontal" H 14600 850 50  0001 C CNN
 F 3 "~" H 14600 850 50  0001 C CNN
 	1    14600 850
@@
 F 0 "J1" H 13580 3942 50  0000 L CNN
 F 1 "Screw_Terminal_01x04" H 13580 3851 50  0000 L CNN
-F 2 "Connector_Phoenix_MSTB:PhoenixContact_MSTBVA_2,5_4-G-5,08_1x04_P5.08mm_Vertical" H 13500 3950 50  0001 C CNN
+F 2 "TerminalBlock_Phoenix:TerminalBlock_Phoenix_MKDS-3-4-5.08_1x04_P5.08mm_Horizontal" H 13500 3950 50  0001 C CNN
 F 3 "~" H 13500 3950 50  0001 C CNN
 	1    13500 3950
@@
 F 0 "J2" H 14230 6142 50  0000 L CNN
 F 1 "Screw_Terminal_01x02" H 14230 6051 50  0000 L CNN
-F 2 "Connector_Phoenix_MSTB:PhoenixContact_MSTBVA_2,5_2-G-5,08_1x02_P5.08mm_Vertical" H 14150 6150 50  0001 C CNN
+F 2 "TerminalBlock_Phoenix:TerminalBlock_Phoenix_MKDS-3-2-5.08_1x02_P5.08mm_Horizontal" H 14150 6150 50  0001 C CNN
 F 3 "~" H 14150 6150 50  0001 C CNN
 	1    14150 6150
@@
 F 0 "J5" H 1430 8692 50  0000 L CNN
 F 1 "Screw_Terminal_01x04" H 1430 8601 50  0000 L CNN
-F 2 "Connector_Phoenix_MSTB:PhoenixContact_MSTBVA_2,5_4-G-5,08_1x04_P5.08mm_Vertical" H 1350 8700 50  0001 C CNN
+F 2 "TerminalBlock_Phoenix:TerminalBlock_Phoenix_MKDS-3-4-5.08_1x04_P5.08mm_Horizontal" H 1350 8700 50  0001 C CNN
 F 3 "~" H 1350 8700 50  0001 C CNN
 	1    1350 8700

Commit message: Finalisation of the Project
Correcte last problems
Create gerber files
Parts:
- C1: footprint Capacitor_SMD:C_1206_3216Metric_Pad1.42x1.75mm_HandSolder -> Capacitor_SMD:CP_Elec_10x12.5
Other:
- note added: "5V PWM CPU Fan"
- note added: "NMEA0183 to Serial"
- note added: "NMEA2000 to SPI"
- note added: "Power management\n9-36V to 5V up to 8A"
- note added: "Real Time Clock"
- moved on the sheet: C11, C12, C13, C23, C24, C25, C5, C7, D1, J2, J5, R1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
