File: Mimosa-Power-Hat.sch (KiCad schematic (older format))
At the start: 74 parts, among them J1 Screw_Terminal_01x04, J2 Screw_Terminal_01x02, J3 40HAT, J4 Screw_Terminal_01x02, J5 Screw_Terminal_01x04, J9 CONN_01X02, M1 Fan_Tacho_PWM, Q1 DMG2305UX, Q2 DMMT5401, U1 ADM3490ExR, U2 CAT24C32, U3 TCAN330, U4 LMZ13608, U5 AB0805, U6 MCP2515-xSO, U7 TXB0102DCU, Y1 32.768 kHz, Y2 8MHz

Commit message: Correction of silk postion of Q1 and Q2
Parts:
- C1: symbol Device:CP -> Mimosa-Power-Hat-rescue:CP-Device
- D1: symbol Device:D_TVS_x2_AAC -> Mimosa-Power-Hat-rescue:D_TVS_x2_AAC-Device
Changed lines of the file:
@@
 $EndComp
 $Comp
-L Device:CP C1
+L Mimosa-Power-Hat-rescue:CP-Device C1
 U 1 1 5EC20D90
 P 9700 1750
@@
 $EndComp
 $Comp
-L Device:D_TVS_x2_AAC D1
+L Mimosa-Power-Hat-rescue:D_TVS_x2_AAC-Device D1
 U 1 1 5ECE214A
 P 14500 6150
